File: HW/Open-Jammer-V1.0/USB.kicad_sch (KiCad schematic)
At the start: 3 parts, among them J2 TYPE-C-31-M-12

Commit message: Added reset and boot buttons. Added oled screen. Added ESP32 VCC capacitors
Other:
- title: (none) -> Oper Jammer V1R0
Changed lines of the file:
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@@
 	(generator_version "9.0")
 	(paper "A5")
+	(title_block
+		(title "Oper Jammer V1R0")
+		(rev "V1R0")
+	)
 	(junction
 		(at 119.38 71.12)
